Commit message: 1

File: src/mobile_robot/urdf/13-diffdrive.urdf.xacro (robot description, xacro)
@@ -1,291 +1,300 @@
 <?xml version="1.0"?>
 <robot name="roscontrol" xmlns:xacro="http://ros.org/wiki/xacro">
-  <xacro:property name="width" value="0.2" />
-  <xacro:property name="leglen" value="0.6" />
-  <xacro:property name="polelen" value="0.2" />
-  <xacro:property name="bodylen" value="0.6" />
-  <xacro:property name="baselen" value="0.4" />
-  <xacro:property name="wheeldiam" value="0.07" />
-  <xacro:property name="pi" value="3.1415" />
-  <material name="blue">
-    <color rgba="0 0 0.8 1"/>
-  </material>
-  <material name="black">
-    <color rgba="0 0 0 1"/>
-  </material>
-  <material name="white">
-    <color rgba="1 1 1 1"/>
-  </material>
-  <xacro:macro name="default_inertial" params="mass">
-    <inertial>
-      <mass value="${mass}" />
-      <inertia ixx="1.0" ixy="0.0" ixz="0.0" iyy="1.0" iyz="0.0" izz="1.0" />
-    </inertial>
-  </xacro:macro>
-  <link name="base_link">
-    <visual>
-      <geometry>
-        <cylinder radius="${width}" length="${bodylen}"/>
-      </geometry>
-      <material name="blue"/>
-    </visual>
-    <collision>
-      <geometry>
-        <cylinder radius="${width}" length="${bodylen}"/>
-      </geometry>
-    </collision>
-    <xacro:default_inertial mass="10"/>
-  </link>
-  <xacro:macro name="wheel" params="prefix suffix reflect">
-    <link name="${prefix}_${suffix}_wheel">
-      <visual>
-        <origin xyz="0 0 0" rpy="${pi/2} 0 0" />
-        <geometry>
-          <cylinder radius="${wheeldiam/2}" length="0.1"/>
-        </geometry>
-        <material name="black"/>
-      </visual>
-      <collision>
-        <origin xyz="0 0 0" rpy="${pi/2} 0 0" />
-        <geometry>
-          <cylinder radius="${wheeldiam/2}" length="0.1"/>
-        </geometry>
-      </collision>
-      <xacro:default_inertial mass="1"/>
+    <xacro:property name="robot_length" value="0.6"/>
+    <xacro:property name="robot_width" value="0.3"/>
+    <xacro:property name="robot_height" value="0.3"/>
+    <xacro:property name="leglen" value="0.6"/>
+    <xacro:property name="polelen" value="0.2"/>
+    <xacro:property name="bodylen" value="0.6"/>
+    <xacro:property name="baselen" value="0.4"/>
+    <xacro:property name="wheeldiam" value="0.15"/>
+    <xacro:property name="pi" value="3.1415"/>
+    <material name="blue">
+        <color rgba="0 0 0.8 1"/>
+    </material>
+    <material name="black">
+        <color rgba="0 0 0 1"/>
+    </material>
+    <material name="white">
+        <color rgba="1 1 1 1"/>
+    </material>
+    <xacro:macro name="default_inertial" params="mass">
+        <inertial>
+            <mass value="${mass}"/>
+            <inertia ixx="1.0" ixy="0.0" ixz="0.0" iyy="1.0" iyz="0.0" izz="1.0"/>
+        </inertial>
+    </xacro:macro>
+    <link name="base_link">
+        <visual>
+            <geometry>
+                <box size="${robot_length} ${robot_width} ${robot_height}"/>
+            </geometry>
+            <material name="blue"/>
+        </visual>
+        <collision>
+            <geometry>
+                <box size="${robot_length} ${robot_width} ${robot_height}"/>
+            </geometry>
+        </collision>
+        <xacro:default_inertial mass="10"/>
     </link>
-    <joint name="${prefix}_${suffix}_wheel_joint" type="continuous">
-      <axis xyz="0 1 0" rpy="0 0 0" />
-      <parent link="${prefix}_base"/>
-      <child link="${prefix}_${suffix}_wheel"/>
-      <origin xyz="${baselen*reflect/3} 0 -${wheeldiam/2+.05}" rpy="0 0 0"/>
-    </joint>
-    <!-- This block provides the simulator (Gazebo) with information on a few additional
-    physical properties. See http://gazebosim.org/tutorials/?tut=ros_urdf for more-->
-    <gazebo reference="${prefix}_${suffix}_wheel">
-      <mu1 value="200.0"/>
-      <mu2 value="100.0"/>
-      <kp value="10000000.0" />
-      <kd value="1.0" />
-      <material>Gazebo/Grey</material>
+    <xacro:macro name="wheel" params="prefix suffix x_reflect y_reflect">
+        <link name="${prefix}_${suffix}_wheel">
+            <visual>
+                <origin xyz="0 0 0" rpy="${pi/2} 0 0"/>
+                <geometry>
+                    <cylinder radius="${wheeldiam/2}" length="0.1"/>
+                </geometry>
+                <material name="black"/>
+            </visual>
+            <collision>
+                <origin xyz="0 0 0" rpy="${pi/2} 0 0"/>
+                <geometry>
+                    <cylinder radius="${wheeldiam/2}" length="0.1"/>
+                </geometry>
+            </collision>
+            <xacro:default_inertial mass="1"/>
+        </link>
+        <joint name="${prefix}_${suffix}_wheel_joint" type="continuous">
+            <axis xyz="1 0 0" rpy="0 0 0"/>
+            <parent link="base_link"/>
+            <child link="${prefix}_${suffix}_wheel"/>
+            <origin xyz="${baselen*x_reflect/3*1.5} ${0.2*y_reflect} -${wheeldiam/2+.05}" rpy="0 0 0"/>
+        </joint>
+        <!-- This block provides the simulator (Gazebo) with information on a few additional
+        physical properties. See http://gazebosim.org/tutorials/?tut=ros_urdf for more-->
+        <gazebo reference="${prefix}_${suffix}_wheel">
+            <mu1 value="200.0"/>
+            <mu2 value="100.0"/>
+            <kp value="10000000.0"/>
+            <kd value="1.0"/>
+            <material>Gazebo/Grey</material>
+        </gazebo>
+        <!-- This block connects the wheel joint to an actuator (motor), which informs both
+        simulation and visualization of the robot -->
+<!--        <transmission name="${prefix}_${suffix}_wheel_trans">-->
+<!--            <type>transmission_interface/SimpleTransmission</type>-->
+<!--            <actuator name="${prefix}_${suffix}_wheel_motor">-->
+<!--                <mechanicalReduction>1</mechanicalReduction>-->
+<!--            </actuator>-->
+<!--            <joint name="${prefix}_${suffix}_wheel_joint">-->
+<!--                <hardwareInterface>VelocityJointInterface</hardwareInterface>-->
+<!--            </joint>-->
+<!--        </transmission>-->
+    </xacro:macro>
+    <xacro:wheel prefix="left" suffix="front" x_reflect="1" y_reflect="1"/>
+    <xacro:wheel prefix="right" suffix="front" x_reflect="-1" y_reflect="1"/>
+    <xacro:wheel prefix="left" suffix="back" x_reflect="1" y_reflect="-1"/>
+    <xacro:wheel prefix="right" suffix="back" x_reflect="-1" y_reflect="-1"/>
+    <xacro:macro name="leg" params="prefix reflect">
+        <link name="${prefix}_leg">
+            <visual>
+                <geometry>
+                    <box size="${leglen} 0.1 0.2"/>
+                </geometry>
+                <origin xyz="0 0 -${leglen/2}" rpy="0 ${pi/2} 0"/>
+                <material name="white"/>
+            </visual>
+            <collision>
+                <geometry>
+                    <box size="${leglen} 0.1 0.2"/>
+                </geometry>
+                <origin xyz="0 0 -${leglen/2}" rpy="0 ${pi/2} 0"/>
+            </collision>
+            <xacro:default_inertial mass="10"/>
+        </link>
+        <joint name="base_to_${prefix}_leg" type="fixed">
+            <parent link="base_link"/>
+            <child link="${prefix}_leg"/>
+            <origin xyz="0 ${reflect*(width+.02)} 0.25"/>
+        </joint>
+        <link name="${prefix}_base">
+            <visual>
+                <geometry>
+                    <box size="${baselen} 0.1 0.1"/>
+                </geometry>
+                <material name="white"/>
+            </visual>
+            <collision>
+                <geometry>
+                    <box size="${baselen} 0.1 0.1"/>
+                </geometry>
+            </collision>
+            <xacro:default_inertial mass="10"/>
+        </link>
+        <joint name="${prefix}_base_joint" type="fixed">
+            <parent link="${prefix}_leg"/>
+            <child link="${prefix}_base"/>
+            <origin xyz="0 0 ${-leglen}"/>
+        </joint>
+        <xacro:wheel prefix="${prefix}" suffix="front" reflect="1"/>
+        <xacro:wheel prefix="${prefix}" suffix="back" reflect="-1"/>
+    </xacro:macro>
+    <!--    <xacro:leg prefix="right" reflect="-1"/>-->
+    <!--    <xacro:leg prefix="left" reflect="1"/>-->
+    <!--    <joint name="gripper_extension" type="prismatic">-->
+    <!--        <parent link="base_link"/>-->
+    <!--        <child link="gripper_pole"/>-->
+    <!--        <limit effort="1000.0" lower="-${width*2-.02}" upper="0" velocity="0.5"/>-->
+    <!--        <origin rpy="0 0 0" xyz="${width-.01} 0 0.2"/>-->
+    <!--        <limit effort="30" velocity="0.2"/>-->
+    <!--        <dynamics damping="0.0" friction="0.0"/>-->
+    <!--    </joint>-->
+    <!--    <link name="gripper_pole">-->
+    <!--        <visual>-->
+    <!--            <geometry>-->
+    <!--                <cylinder length="${polelen}" radius="0.01"/>-->
+    <!--            </geometry>-->
+    <!--            <origin xyz="${polelen/2} 0 0" rpy="0 ${pi/2} 0 "/>-->
+    <!--        </visual>-->
+    <!--        <collision>-->
+    <!--            <geometry>-->
+    <!--                <cylinder length="${polelen}" radius="0.01"/>-->
+    <!--            </geometry>-->
+    <!--            <origin xyz="${polelen/2} 0 0" rpy="0 ${pi/2} 0 "/>-->
+    <!--        </collision>-->
+    <!--        <xacro:default_inertial mass="0.05"/>-->
+    <!--    </link>-->
+    <!--    <transmission name="gripper_extension_trans">-->
+    <!--        <type>transmission_interface/SimpleTransmission</type>-->
+    <!--        <actuator name="gripper_extension_motor">-->
+    <!--            <mechanicalReduction>1</mechanicalReduction>-->
+    <!--        </actuator>-->
+    <!--        <joint name="gripper_extension">-->
+    <!--            <hardwareInterface>PositionJointInterface</hardwareInterface>-->
+    <!--        </joint>-->
+    <!--    </transmission>-->
+    <xacro:macro name="gripper" params="prefix reflect">
+        <joint name="${prefix}_gripper_joint" type="revolute">
+            <axis xyz="0 0 ${reflect}"/>
+            <limit effort="1000.0" lower="0.0" upper="0.548" velocity="0.5"/>
+            <origin rpy="0 0 0" xyz="${polelen} ${reflect*0.01} 0"/>
+            <parent link="gripper_pole"/>
+            <child link="${prefix}_gripper"/>
+            <limit effort="30" velocity="1.0"/>
+            <dynamics damping="0.0" friction="0.0"/>
+        </joint>
+        <link name="${prefix}_gripper">
+            <visual>
+                <origin rpy="${(reflect-1)/2*pi} 0 0" xyz="0 0 0"/>
+                <geometry>
+                    <mesh filename="package://urdf_tutorial/meshes/l_finger.dae"/>
+                </geometry>
+            </visual>
+            <collision>
+                <geometry>
+                    <mesh filename="package://urdf_tutorial/meshes/l_finger.dae"/>
+                </geometry>
+                <origin rpy="${(reflect-1)/2*pi} 0 0" xyz="0 0 0"/>
+            </collision>
+            <xacro:default_inertial mass="0.05"/>
+        </link>
+        <transmission name="${prefix}_gripper_trans">
+            <type>transmission_interface/SimpleTransmission</type>
+            <actuator name="${prefix}_gripper_motor">
+                <mechanicalReduction>1</mechanicalReduction>
+            </actuator>
+            <joint name="${prefix}_gripper_joint">
+                <hardwareInterface>PositionJointInterface</hardwareInterface>
+            </joint>
+        </transmission>
+        <joint name="${prefix}_tip_joint" type="fixed">
+            <parent link="${prefix}_gripper"/>
+            <child link="${prefix}_tip"/>
+        </joint>
+        <link name="${prefix}_tip">
+            <visual>
+                <origin rpy="${(reflect-1)/2*pi} 0 0" xyz="0.09137 0.00495 0"/>
+                <geometry>
+                    <mesh filename="package://urdf_tutorial/meshes/l_finger_tip.dae"/>
+                </geometry>
+            </visual>
+            <collision>
+                <geometry>
+                    <mesh filename="package://urdf_tutorial/meshes/l_finger_tip.dae"/>
+                </geometry>
+                <origin rpy="${(reflect-1)/2*pi} 0 0" xyz="0.09137 0.00495 0"/>
+            </collision>
+            <xacro:default_inertial mass="0.05"/>
+        </link>
+    </xacro:macro>
+    <!--    <xacro:gripper prefix="left" reflect="1"/>-->
+    <!--    <xacro:gripper prefix="right" reflect="-1"/>-->
+    <!--    <link name="head">-->
+    <!--        <visual>-->
+    <!--            <geometry>-->
+    <!--                <sphere radius="${width}"/>-->
+    <!--            </geometry>-->
+    <!--            <material name="white"/>-->
+    <!--        </visual>-->
+    <!--        <collision>-->
+    <!--            <geometry>-->
+    <!--                <sphere radius="${width}"/>-->
+    <!--            </geometry>-->
+    <!--        </collision>-->
+    <!--        <xacro:default_inertial mass="2"/>-->
+    <!--    </link>-->
+    <!--    <joint name="head_swivel" type="continuous">-->
+    <!--        <parent link="base_link"/>-->
+    <!--        <child link="head"/>-->
+    <!--        <axis xyz="0 0 1"/>-->
+    <!--        <origin xyz="0 0 ${bodylen/2}"/>-->
+    <!--        <limit effort="30" velocity="1.0"/>-->
+    <!--        <dynamics damping="0.0" friction="0.0"/>-->
+    <!--    </joint>-->
+    <!-- This block connects the head_swivel joint to an actuator (motor), which informs both
+    simulation and visualization of the robot -->
+    <!--    <transmission name="head_swivel_trans">-->
+    <!--        <type>transmission_interface/SimpleTransmission</type>-->
+    <!--        <actuator name="$head_swivel_motor">-->
+    <!--            <mechanicalReduction>1</mechanicalReduction>-->
+    <!--        </actuator>-->
+    <!--        <joint name="head_swivel">-->
+    <!--            <hardwareInterface>PositionJointInterface</hardwareInterface>-->
+    <!--        </joint>-->
+    <!--    </transmission>-->
+    <!--    <link name="box">-->
+    <!--        <visual>-->
+    <!--            <geometry>-->
+    <!--                <box size="0.08 0.08 0.08"/>-->
+    <!--            </geometry>-->
+    <!--            <material name="blue"/>-->
+    <!--            <origin xyz="-0.04 0 0"/>-->
+    <!--        </visual>-->
+    <!--        <collision>-->
+    <!--            <geometry>-->
+    <!--                <box size="0.08 0.08 0.08"/>-->
+    <!--            </geometry>-->
+    <!--        </collision>-->
+    <!--        <xacro:default_inertial mass="1"/>-->
+    <!--    </link>-->
+    <!--    <joint name="tobox" type="fixed">-->
+    <!--        <parent link="head"/>-->
+    <!--        <child link="box"/>-->
+    <!--        <origin xyz="${.707*width+0.04} 0 ${.707*width}"/>-->
+    <!--    </joint>-->
+    <!-- Gazebo plugin for ROS Control -->
+    <gazebo>
+        <plugin name="gazebo_ros_control" filename="libgazebo_ros_control.so">
+            <robotNamespace>/</robotNamespace>
+        </plugin>
     </gazebo>
-    <!-- This block connects the wheel joint to an actuator (motor), which informs both
-    simulation and visualization of the robot -->
-    <transmission name="${prefix}_${suffix}_wheel_trans">
-      <type>transmission_interface/SimpleTransmission</type>
-      <actuator name="${prefix}_${suffix}_wheel_motor">
-        <mechanicalReduction>1</mechanicalReduction>
-      </actuator>
-      <joint name="${prefix}_${suffix}_wheel_joint">
-        <hardwareInterface>VelocityJointInterface</hardwareInterface>
-      </joint>
-    </transmission>
-  </xacro:macro>
-  <xacro:macro name="leg" params="prefix reflect">
-    <link name="${prefix}_leg">
-      <visual>
-        <geometry>
-          <box size="${leglen} 0.1 0.2"/>
-        </geometry>
-        <origin xyz="0 0 -${leglen/2}" rpy="0 ${pi/2} 0"/>
-        <material name="white"/>
-      </visual>
-      <collision>
-        <geometry>
-          <box size="${leglen} 0.1 0.2"/>
-        </geometry>
-        <origin xyz="0 0 -${leglen/2}" rpy="0 ${pi/2} 0"/>
-      </collision>
-      <xacro:default_inertial mass="10"/>
-    </link>
-    <joint name="base_to_${prefix}_leg" type="fixed">
-      <parent link="base_link"/>
-      <child link="${prefix}_leg"/>
-      <origin xyz="0 ${reflect*(width+.02)} 0.25" />
-    </joint>
-    <link name="${prefix}_base">
-      <visual>
-        <geometry>
-          <box size="${baselen} 0.1 0.1"/>
-        </geometry>
-        <material name="white"/>
-      </visual>
-      <collision>
-        <geometry>
-          <box size="${baselen} 0.1 0.1"/>
-        </geometry>
-      </collision>
-      <xacro:default_inertial mass="10"/>
-    </link>
-    <joint name="${prefix}_base_joint" type="fixed">
-      <parent link="${prefix}_leg"/>
-      <child link="${prefix}_base"/>
-      <origin xyz="0 0 ${-leglen}" />
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
Commit message: xd

File: src/mobile_robot/urdf/13-diffdrive.urdf.xacro (robot description, xacro)
@@ -57,5 +57,5 @@
         </link>
         <joint name="${prefix}_${suffix}_wheel_joint" type="continuous">
-            <axis xyz="1 0 0" rpy="0 0 0"/>
+            <axis xyz="0 1 0" rpy="0 0 0"/>
             <parent link="base_link"/>
             <child link="${prefix}_${suffix}_wheel"/>
@@ -73,17 +73,17 @@
         <!-- This block connects the wheel joint to an actuator (motor), which informs both
         simulation and visualization of the robot -->
-<!--        <transmission name="${prefix}_${suffix}_wheel_trans">-->
-<!--            <type>transmission_interface/SimpleTransmission</type>-->
-<!--            <actuator name="${prefix}_${suffix}_wheel_motor">-->
-<!--                <mechanicalReduction>1</mechanicalReduction>-->
-<!--            </actuator>-->
-<!--            <joint name="${prefix}_${suffix}_wheel_joint">-->
-<!--                <hardwareInterface>VelocityJointInterface</hardwareInterface>-->
-<!--            </joint>-->
-<!--        </transmission>-->
+       <transmission name="${prefix}_${suffix}_wheel_trans">
+           <type>transmission_interface/SimpleTransmission</type>
+           <actuator name="${prefix}_${suffix}_wheel_motor">
+               <mechanicalReduction>1</mechanicalReduction>
+           </actuator>
+           <joint name="${prefix}_${suffix}_wheel_joint">
+               <hardwareInterface>VelocityJointInterface</hardwareInterface>
+           </joint>
+       </transmission>
     </xacro:macro>
     <xacro:wheel prefix="left" suffix="front" x_reflect="1" y_reflect="1"/>
-    <xacro:wheel prefix="right" suffix="front" x_reflect="-1" y_reflect="1"/>
-    <xacro:wheel prefix="left" suffix="back" x_reflect="1" y_reflect="-1"/>
+    <xacro:wheel prefix="right" suffix="front" x_reflect="1" y_reflect="-1"/>
+    <xacro:wheel prefix="left" suffix="back" x_reflect="-1" y_reflect="1"/>
     <xacro:wheel prefix="right" suffix="back" x_reflect="-1" y_reflect="-1"/>
     <xacro:macro name="leg" params="prefix reflect">

Commit message: xd1

File: src/mobile_robot/urdf/13-diffdrive.urdf.xacro (robot description, xacro)
@@ -37,6 +37,27 @@
             </geometry>
         </collision>
-        <xacro:default_inertial mass="10"/>
+        <!-- <xacro:default_inertial mass="10"/> -->
     </link>
+    <link name="dummy_base_link">
+        <!-- <visual>
+            <geometry>
+                <origin xyz="0 0 0" rpy="0 0 0"/>
+                <box size="${robot_length} ${robot_width} ${robot_height}"/>
+            </geometry>
+            <material name="blue"/>
+        </visual>
+        <collision>
+            <geometry>
+                <origin xyz="0 0 0" rpy="0 0 0"/>
+                <box size="${robot_length} ${robot_width} ${robot_height}"/>
+            </geometry>
+        </collision> -->
+        <xacro:default_inertial mass="20"/>
+    </link>
+    <joint name="dummy_joint" type="fixed">
+        <parent link="base_link"/>
+        <child link="dummy_base_link"/>
+        <origin xyz="0 0 0 " rpy="0 0 0"/>
+    </joint>
     <xacro:macro name="wheel" params="prefix suffix x_reflect y_reflect">
         <link name="${prefix}_${suffix}_wheel">
@@ -79,5 +100,5 @@
            </actuator>
            <joint name="${prefix}_${suffix}_wheel_joint">
-               <hardwareInterface>VelocityJointInterface</hardwareInterface>
+               <hardwareInterface>hardware_interface/VelocityJointInterface</hardwareInterface>
            </joint>
        </transmission>
